File: hardware/pd_board/pd_board.kicad_pcb (KiCad board)
At the start: 2 copper layers, 53.6 x 35.6 mm, 51 parts, among them J1 USB_C_Receptacle_USB2.0_16P, J2 Dead_Battery_CC1, J3 Dead_Battery_CC2, J4 Debug Port, J5 UART_Port, U1 FUSB302BMPX, U2 TPS5420D, U3 STM32F072CBUx

Commit message: update
Routing:
- net /INT_N: track 27.5 -> 25.0 mm
Other:
- board text added: "BOOT"
Changed lines of the file:
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@@
 			(psa4output no)
 			(plot_black_and_white yes)
-			(plotinvisibletext no)
 			(sketchpadsonfab no)
 			(plotpadnumbers no)
@@
 			)
 		)
-		(property "Datasheet" ""
+		(property "Datasheet" "~"
 			(at 0 0 180)
 			(unlocked yes)
@@
 			)
 		)
-		(property "Datasheet" ""
+		(property "Datasheet" "~"
 			(at 0 0 180)
 			(unlocked yes)
@@
 			)
 		)
-		(property "Datasheet" ""
+		(property "Datasheet" "~"
 			(at 0 0 0)
 			(unlocked yes)
@@
 			)
 		)
-		(property "Datasheet" ""
+		(property "Datasheet" "~"
 			(at 0 0 0)
 			(unlocked yes)
@@
 			)
 		)
-		(property "Datasheet" ""
+		(property "Datasheet" "~"
 			(at 0 0 90)
 			(layer "F.Fab")
@@
 			)
 		)
-		(property "Datasheet" ""
+		(property "Datasheet" "~"
 			(at 0 0 90)
 			(layer "F.Fab")
@@
 			)
 		)
-		(property "Datasheet" ""
+		(property "Datasheet" "~"
 			(at 0 0 270)
 			(unlocked yes)
@@
 			)
 		)
-		(property "Datasheet" ""
+		(property "Datasheet" "~"
 			(at 0 0 0)
 			(unlocked yes)
@@
 			)
 		)
-		(property "Datasheet" ""
+		(property "Datasheet" "~"
 			(at 0 0 180)
 			(unlocked yes)
@@
 			)
 		)
-		(property "Datasheet" ""
+		(property "Datasheet" "~"
 			(at 0 0 90)
 			(unlocked yes)
@@
 			)
 		)
-		(property "Datasheet" ""
+		(property "Datasheet" "~"
 			(at 0 0 0)
 			(layer "F.Fab")
@@
 			)
 		)
-		(property "Datasheet" ""
+		(property "Datasheet" "~"
 			(at 0 0 180)
 			(unlocked yes)
@@
 			)
 		)
-		(property "Datasheet" ""
+		(property "Datasheet" "~"
 			(at 0 0 0)
 			(unlocked yes)
@@
 			)
 		)
-		(property "Datasheet" ""
+		(property "Datasheet" "~"
 			(at 0 0 90)
 			(layer "F.Fab")
@@
 			)
 		)
-		(property "Datasheet" ""
+		(property "Datasheet" "~"
 			(at 0 0 180)
 			(unlocked yes)
@@
 			)
 		)
-		(property "Datasheet" ""
+		(property "Datasheet" "~"
 			(at 0 0 180)
 			(unlocked yes)
@@
 			)
 		)
-		(property "Datasheet" ""
+		(property "Datasheet" "~"
 			(at 0 0 0)
 			(unlocked yes)
@@
 			)
 		)
-		(property "Datasheet" ""
+		(property "Datasheet" "~"
 			(at 0 0 0)
 			(unlocked yes)
@@
 			)
 		)
-		(property "Datasheet" ""
+		(property "Datasheet" "~"
 			(at 0 0 180)
 			(unlocked yes)
@@
 			)
 		)
-		(property "Datasheet" ""
+		(property "Datasheet" "~"
 			(at 0 0 0)
 			(unlocked yes)
@@
 			)
 		)
-		(property "Datasheet" ""
+		(property "Datasheet" "~"
 			(at 0 0 90)
 			(unlocked yes)
@@
 			)
 		)
-		(property "Datasheet" ""
+		(property "Datasheet" "~"
 			(at 0 0 0)
 			(unlocked yes)
@@
 			)
 		)
-		(property "Datasheet" ""
+		(property "Datasheet" "~"
 			(at 0 0 180)
 			(unlocked yes)
@@
 			)
 		)
-		(property "Datasheet" ""
+		(property "Datasheet" "~"
 			(at 0 0 180)
 			(unlocked yes)
@@
 			)
 		)
-		(property "Datasheet" ""
+		(property "Datasheet" "~"
 			(at 0 0 270)
 			(unlocked yes)
@@
 			)
 		)
-		(property "Datasheet" ""
+		(property "Datasheet" "~"
 			(at 0 0 0)
 			(unlocked yes)
@@
 			)
 		)
-		(property "Datasheet" ""
+		(property "Datasheet" "~"
 			(at 0 0 90)
 			(layer "F.Fab")
@@
 			)
 		)
-		(property "Datasheet" ""
+		(property "Datasheet" "~"
 			(at 0 0 0)
 			(unlocked yes)
@@
 			)
 		)
-		(property "Datasheet" ""
+		(property "Datasheet" "~"
 			(at 0 0 90)
 			(unlocked yes)
@@
 			)
 		)
-		(property "Datasheet" ""
+		(property "Datasheet" "~"
 			(at 0 0 270)
 			(unlocked yes)
@@
 			)
 		)
-		(property "Datasheet" ""
+		(property "Datasheet" "~"
 			(at 0 0 0)
 			(unlocked yes)
@@
 			)
 		)
-		(property "Datasheet" ""
+		(property "Datasheet" "~"
 			(at 0 0 270)
 			(unlocked yes)
@@
 			)
 		)
-		(property "Datasheet" ""
+		(property "Datasheet" "~"
 			(at 0 0 0)
 			(unlocked yes)
@@
 			)
 		)
-		(property "Datasheet" ""
+		(property "Datasheet" "~"
 			(at 0 0 0)
 			(layer "F.Fab")
@@
 			)
 		)
-		(property "Datasheet" ""
+		(property "Datasheet" "~"
 			(at 0 0 90)
 			(unlocked yes)
@@
 			)
 		)
-		(property "Datasheet" ""
+		(property "Datasheet" "~"
 			(at 0 0 270)
 			(unlocked yes)
@@
 			)
 		)
-		(property "Datasheet" ""
+		(property "Datasheet" "~"
 			(at 0 0 0)
 			(unlocked yes)
@@
 			)
 		)
-		(property "Datasheet" ""
+		(property "Datasheet" "~"
 			(at 0 0 0)
 			(unlocked yes)
@@
 			)
 		)
-		(property "Datasheet" ""
+		(property "Datasheet" "~"
 			(at 0 0 0)
 			(unlocked yes)
@@
 			)
 		)
-		(property "Datasheet" ""
+		(property "Datasheet" "~"
 			(at 0 0 270)
 			(unlocked yes)
@@
 			)
 		)
-		(property "Datasheet" ""
+		(property "Datasheet" "~"
 			(at 0 0 90)
 			(unlocked yes)
@@
 			)
 		)
-		(property "Datasheet" ""
+		(property "Datasheet" "~"
 			(at 0 0 0)
 			(unlocked yes)
@@
 		)
 	)
+	(gr_text "BOOT"
+		(at 148.4 75.6 0)
+		(layer "F.SilkS")
+		(effects
+			(font
+				(size 0.5 0.5)
+				(thickness 0.1)
+				(bold yes)
+			)
+			(justify left bottom)
+		)
+	)
 	(gr_text "GND"
 		(at 155.5 108.5 0)
@@
 	)
 	(segment
-		(start 124.9279 89.4467)
-		(end 124.308 89.4467)
-		(width 0.2)
-		(layer "F.Cu")
-		(net 23)
-	)
-	(segment
-		(start 124.308 89.4467)
-		(end 124.9279 89.4467)
-		(width 0.2)
-		(layer "F.Cu")
-		(net 23)
-	)
-	(segment
 		(start 122.042 90.3065)
 		(end 122.1282 90.3927)
@@
 	)
 	(segment
-		(start 122.8469 89.674)
-		(end 122.1282 90.3927)
+		(start 124.9279 89.4467)
+		(end 122.847 89.4467)
 		(width 0.2)
 		(layer "B.Cu")
@@
 	)
 	(segment
-		(start 124.308 89.4467)
-		(end 124.9279 89.4467)
+		(start 122.8469 89.674)
+		(end 122.1282 90.3927)
 		(width 0.2)
 		(layer "B.Cu")
@@
 		(width 0.2)
 		(layer "B.Cu")
-		(net 23)
-	)
-	(segment
-		(start 124.9279 89.4467)
-		(end 124.308 89.4467)
-		(width 0.2)
-		(layer "B.Cu")
-		(net 23)
-	)
-	(segment
-		(start 124.9279 89.4467)
-		(end 122.847 89.4467)
-		(width 0.2)
-		(layer "B.Cu")

Commit message: update
Parts:
- removed TP1: CC2_TP, TestPoint:TestPoint_Pad_1.0x1.0mm
- removed TP2: VCONN_TP, TestPoint:TestPoint_Pad_1.0x1.0mm
- removed TP3: CC1_TP, TestPoint:TestPoint_Pad_1.0x1.0mm
- removed TP4: GND_TP, TestPoint:TestPoint_Pad_1.0x1.0mm
- added J6: VBUS_JP, Connector_PinHeader_2.54mm:PinHeader_1x02_P2.54mm_Vertical, F.Cu at (113.2, 77.3)
- added J7: VCONN_JP, Connector_PinHeader_2.54mm:PinHeader_1x02_P2.54mm_Vertical, F.Cu at (117.8, 77.3)
- moved R3 0.23 mm to (136.6, 86.4)
- moved R2 0.23 mm to (138.0, 86.3)
- moved FB1 0.22 mm to (140.8, 83.0)
- moved C10 0.20 mm to (141.8, 86.2)
- moved C2 0.20 mm to (139.8, 86.2)
Connections:
- D4 pad 2: /VBUS_IN -> /VBUS
- D5 pad 1: /VBUS_IN -> +3.3V
- D6 pad 1: /VBUS_IN -> +3.3V
- J1 pad A4: /VBUS_IN -> /VBUS
- J1 pad A9: /VBUS_IN -> /VBUS
- J1 pad B4: /VBUS_IN -> /VBUS
- J1 pad B9: /VBUS_IN -> /VBUS
- U1 pad 2: /VBUS_IN -> /VBUS
Routing:
- net /VBUS_IN: track 62.7 -> 0.00 mm, vias 2 -> 0
- net /VBUS: track 0.00 -> 44.0 mm, vias 0 -> 1
- net /INT_N: track 25.0 -> 60.5 mm, vias 3 -> 2
- net Net-(U3-VDDA): track 22.2 -> 44.8 mm, vias 2 -> 5
- net GND: track 229.8 -> 251.8 mm, vias 7 -> 4
- net /CC2: track 52.2 -> 31.4 mm, vias 0 -> 2
- net +3.3V: track 132.0 -> 152.5 mm, vias 6 -> 4
- net Net-(U2-VSNS): track 26.3 -> 40.8 mm, vias 2 -> 0
- net /CC1: track 37.4 -> 26.7 mm, vias 2 -> 3
- net Net-(U2-PH): track 3.50 -> 11.4 mm, vias 0 -> 2
- net /NRST: track 17.7 -> 11.9 mm, vias 2 -> 0
- net /I2C_SDA: track 21.2 -> 25.0 mm
- net /USB_DN: track 46.6 -> 43.6 mm
- net /BOOT: track 28.6 -> 25.8 mm
- net /SWCLK: track 18.7 -> 16.3 mm
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Other:
- board text added: "CC1"
- board text added: "CC2"
- board text added: "VBUS"
- board text added: "VCONN"
