File: hardware/pd_board/pd_board.kicad_pcb (KiCad board)
At the start: 2 copper layers, 53.6 x 35.6 mm, 49 parts, among them J1 USB_C_Receptacle_USB2.0_16P, J2 Dead_Battery_CC1, J3 Dead_Battery_CC2, J4 Debug Port, J5 UART_Port, J6 VBUS_JP, J7 VCONN_JP, U1 FUSB302BMPX, U2 TPS5420D, U3 STM32F072CBUx

Commit message: update
Parts:
- removed R5, R6: 5.1k, Resistor_SMD:R_0402_1005Metric
- J2: value Dead_Battery_CC1 -> CC1_TP; footprint Connector_PinHeader_2.54mm:PinHeader_1x02_P2.54mm_Vertical -> Connector_PinHeader_2.54mm:PinHeader_1x01_P2.54mm_Vertical
- J3: value Dead_Battery_CC2 -> CC2_TP; footprint Connector_PinHeader_2.54mm:PinHeader_1x02_P2.54mm_Vertical -> Connector_PinHeader_2.54mm:PinHeader_1x01_P2.54mm_Vertical
- moved J4 13.1 mm to (141.8, 95.8)
- moved JP1 11.6 mm to (136.5, 77.2), turned to -90 degrees
- moved J5 10.4 mm to (149.6, 98.0), turned to 180 degrees
- moved C11 5.59 mm to (139.4, 84.5)
- moved C12 5.59 mm to (142.4, 84.5)
- moved C6 5.59 mm to (138.0, 84.5)
- moved C9 5.59 mm to (141.0, 84.5)
- moved D5 5.57 mm to (143.6, 100.8)
- moved C10 5.43 mm to (136.4, 85.2)
- moved C2 5.43 mm to (134.4, 85.2)
- moved C8 5.43 mm to (126.5, 85.0)
- moved R2 5.43 mm to (132.7, 85.4)
- moved R3 5.43 mm to (131.2, 85.5)
- moved R7 5.43 mm to (128.7, 85.0)
- moved U3 5.40 mm to (133.4, 92.8)
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Connections:
- C5 pad 1: /CC2 -> /CC1
- C7 pad 1: /CC1 -> GND
- C7 pad 2: GND -> /CC2
Routing:
- net GND: track 251.8 -> 204.5 mm, vias 4 -> 5
- net /INT_N: track 60.5 -> 23.1 mm, vias 2 -> 3
- net Net-(U3-VDDA): track 44.8 -> 24.6 mm, vias 5 -> 3
- net /CC2: track 31.4 -> 50.2 mm, vias 2 -> 3
- net Net-(U2-VSNS): track 40.8 -> 23.3 mm, vias 0 -> 2
- net /UART_RTS: track 19.8 -> 34.6 mm, vias 0 -> 3
- net /NRST: track 11.9 -> 25.5 mm, vias 0 -> 2
- net /USB_DP: track 41.9 -> 29.2 mm
- net /CC1: track 26.7 -> 36.4 mm, vias 3 -> 1
- net Net-(J2-Pin_2): track 9.07 -> 0.00 mm, vias 1 -> 0
- net +3.3V: track 152.5 -> 143.4 mm, vias 4 -> 5
- net /UART_CTS: track 18.3 -> 26.5 mm, vias 1 -> 0
- net /SWDIO: track 13.3 -> 5.06 mm
- net Net-(U2-PH): track 11.4 -> 3.50 mm, vias 2 -> 0
- net /UART_TX: track 20.4 -> 28.1 mm, vias 0 -> 1
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- added copper zone on B.Cu, net GND
Other:
- board size 53.6 x 35.6 mm -> 48.4 x 35.6 mm

Commit message: update
Parts:
- added J8: VIN_ENA_JP, Connector_PinHeader_2.54mm:PinHeader_1x02_P2.54mm_Vertical, F.Cu at (149.6, 104.2)
Connections:
- net Net-(D3-K) renamed /VIN
- U2 pad 5: unconnected-(U2-ENA-Pad5) -> /VIN_ENA
Routing:
- net /VIN: track 17.0 -> 48.9 mm, vias 0 -> 1
- net /VIN_ENA: track 0.00 -> 30.3 mm, vias 0 -> 1

Commit message: update
Parts:
- removed J8: VIN_ENA_JP, Connector_PinHeader_2.54mm:PinHeader_1x02_P2.54mm_Vertical
Connections:
- C19 pad 1: /VIN -> Net-(D3-K)
- D3 pad 1: /VIN -> Net-(D3-K)
- D4 pad 1: /VIN -> Net-(D3-K)
- U2 pad 5: /VIN_ENA -> Net-(D3-K)
- U2 pad 7: /VIN -> Net-(D3-K)
Routing:
- net /VIN: track 48.9 -> 0.00 mm, vias 1 -> 0
- net /VIN_ENA: track 30.3 -> 0.00 mm, vias 1 -> 0
- net Net-(D3-K): track 0.00 -> 22.1 mm, vias 0 -> 2

Commit message: update
Parts:
- added J8: VIN_ENA_JP, Connector_PinHeader_2.54mm:PinHeader_1x02_P2.54mm_Vertical, F.Cu at (149.6, 104.2)
Connections:
- C19 pad 1: Net-(D3-K) -> /VIN
- D3 pad 1: Net-(D3-K) -> /VIN
- D4 pad 1: Net-(D3-K) -> /VIN
- U2 pad 5: Net-(D3-K) -> /VIN_ENA
- U2 pad 7: Net-(D3-K) -> /VIN
Routing:
- net /VIN: track 0.00 -> 48.9 mm, vias 0 -> 1
- net /VIN_ENA: track 0.00 -> 30.3 mm, vias 0 -> 1
- net Net-(D3-K): track 22.1 -> 0.00 mm, vias 2 -> 0
