File: hardware/pd_board/pd_board.kicad_sch (KiCad schematic)
At the start: 51 parts, among them J1 USB_C_Receptacle_USB2.0_16P, J2 Dead_Battery_CC1, J3 Dead_Battery_CC2, J4 Debug Port, J5 UART_Port, U1 FUSB302BMPX, U2 TPS5420D, U3 STM32F072CBUx

Commit message: update
Other:
- moved on the sheet: R4
Changed lines of the file:
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@@
 	)
 	(junction
-		(at 247.65 30.48)
+		(at 207.01 97.79)
 		(diameter 0)
 		(color 0 0 0 0)
 	)
 	(junction
-		(at 34.29 120.65)
+		(at 247.65 30.48)
 		(diameter 0)
 		(color 0 0 0 0)
 	)
 	(junction
-		(at 35.56 69.85)
+		(at 34.29 120.65)
 		(diameter 0)
 		(color 0 0 0 0)
@@
 	(wire
 		(pts
+			(xy 207.01 82.55) (xy 210.82 82.55)
+		)
+		(stroke
+			(width 0)
+			(type default)
+		)
+	)
+	(wire
+		(pts
 			(xy 34.29 129.54) (xy 34.29 130.81)
 		)
@@
 	(wire
 		(pts
+			(xy 207.01 97.79) (xy 220.98 97.79)
+		)
+		(stroke
+			(width 0)
+			(type default)
+		)
+	)
+	(wire
+		(pts
 			(xy 269.24 41.91) (xy 269.24 44.45)
 		)
@@
 	(wire
 		(pts
-			(xy 142.24 41.91) (xy 149.86 41.91)
+			(xy 210.82 91.44) (xy 210.82 95.25)
 		)
 		(stroke
@@
 	(wire
 		(pts
-			(xy 210.82 91.44) (xy 210.82 95.25)
+			(xy 110.49 121.92) (xy 118.11 121.92)
 		)
 		(stroke
@@
 	(wire
 		(pts
-			(xy 110.49 121.92) (xy 118.11 121.92)
+			(xy 93.98 147.32) (xy 102.87 147.32)
 		)
 		(stroke
@@
 	(wire
 		(pts
-			(xy 93.98 147.32) (xy 102.87 147.32)
+			(xy 82.55 163.83) (xy 82.55 167.64)
 		)
 		(stroke
@@
 	(wire
 		(pts
-			(xy 82.55 163.83) (xy 82.55 167.64)
+			(xy 80.01 121.92) (xy 83.82 121.92)
 		)
 		(stroke
@@
 	(wire
 		(pts
-			(xy 80.01 121.92) (xy 83.82 121.92)
+			(xy 210.82 82.55) (xy 210.82 83.82)
 		)
 		(stroke
@@
 	(wire
 		(pts
-			(xy 210.82 82.55) (xy 210.82 83.82)
+			(xy 69.85 132.08) (xy 69.85 147.32)
 		)
 		(stroke
@@
 	(wire
 		(pts
-			(xy 69.85 132.08) (xy 69.85 147.32)
+			(xy 207.01 82.55) (xy 207.01 83.82)
 		)
 		(stroke
@@
 	(wire
 		(pts
-			(xy 27.94 69.85) (xy 35.56 69.85)
-		)
-		(stroke
-			(width 0)
-			(type default)
-		)
-	)
-	(wire
-		(pts
 			(xy 189.23 50.8) (xy 189.23 49.53)
 		)
@@
 	(wire
 		(pts
-			(xy 157.48 41.91) (xy 160.02 41.91)
-		)
-		(stroke
-			(width 0)
-			(type default)
-		)
-	)
-	(wire
-		(pts
 			(xy 102.87 147.32) (xy 110.49 147.32)
 		)
@@
 	(wire
 		(pts
-			(xy 205.74 97.79) (xy 220.98 97.79)
+			(xy 205.74 97.79) (xy 207.01 97.79)
 		)
 		(stroke
@@
 	(wire
 		(pts
+			(xy 207.01 91.44) (xy 207.01 97.79)
+		)
+		(stroke
+			(width 0)
+			(type default)
+		)
+	)
+	(wire
+		(pts
 			(xy 102.87 147.32) (xy 102.87 156.21)
 		)
@@
 	(wire
 		(pts
+			(xy 142.24 41.91) (xy 148.59 41.91)
+		)
+		(stroke
+			(width 0)
+			(type default)
+		)
+	)
+	(wire
+		(pts
 			(xy 198.12 54.61) (xy 200.66 54.61)
 		)
@@
 	(symbol
 		(lib_id "Device:R")
-		(at 153.67 41.91 90)
+		(at 207.01 87.63 180)
 		(unit 1)
 		(exclude_from_sim no)
@@
 		(dnp no)
 		(property "Reference" "R4"
-			(at 154.178 39.624 90)
+			(at 204.978 84.582 0)
 			(effects
 				(font
@@
 		)
 		(property "Value" "4.7k"
-			(at 153.67 41.91 90)
+			(at 207.01 87.63 90)
 			(effects
 				(font
@@
 		)
 		(property "Footprint" "Resistor_SMD:R_0402_1005Metric"
-			(at 153.67 43.688 90)
+			(at 208.788 87.63 90)
 			(effects
 				(font
@@
 		)
 		(property "Datasheet" "~"
-			(at 153.67 41.91 0)
+			(at 207.01 87.63 0)
 			(effects
 				(font
@@
 		)
 		(property "Description" "Resistor"
-			(at 153.67 41.91 0)
+			(at 207.01 87.63 0)
 			(effects
 				(font
@@
 	)
 	(symbol
-		(lib_id "power:+3.3V")
-		(at 160.02 41.91 0)
-		(unit 1)
-		(exclude_from_sim no)
-		(in_bom yes)
-		(on_board yes)
-		(dnp no)
-		(fields_autoplaced yes)
-		(property "Reference" "#PWR015"
-			(at 160.02 45.72 0)
-			(effects
-				(font
-					(size 1.27 1.27)
-				)
-				(hide yes)
-			)
-		)
-		(property "Value" "+3.3V"
-			(at 160.02 36.83 0)
-			(effects
-				(font
-					(size 1.27 1.27)
-				)
-			)
-		)
-		(property "Footprint" ""
-			(at 160.02 41.91 0)
-			(effects
-				(font
-					(size 1.27 1.27)
-				)
-				(hide yes)
-			)
-		)
-		(property "Datasheet" ""
-			(at 160.02 41.91 0)
-			(effects
-				(font
-					(size 1.27 1.27)
-				)
-				(hide yes)
-			)
-		)
-		(property "Description" "Power symbol creates a global label with name \"+3.3V\""
-			(at 160.02 41.91 0)
-			(effects
-				(font
-					(size 1.27 1.27)
-				)
-				(hide yes)
-			)
-		)
-		(pin "1"
-		)
-		(instances
-			(project ""
-				(path "/9d05689f-cd28-4719-8892-8398308a18b8"
-					(reference "#PWR015")
-					(unit 1)
-				)
-			)
-		)
-	)
-	(symbol
 		(lib_id "Device:C_Small")
 		(at 34.29 127 0)
@@
 					(unit 1)
 				)
+			)
+		)
+	)
+	(symbol
+		(lib_id "power:GND")
+		(at 27.94 69.85 0)
+		(unit 1)
+		(exclude_from_sim no)
+		(in_bom yes)
+		(on_board yes)
+		(dnp no)
+		(fields_autoplaced yes)
+		(property "Reference" "#PWR010"
+			(at 27.94 76.2 0)
+			(effects
+				(font
+					(size 1.27 1.27)
+				)
+				(hide yes)
+			)
+		)
+		(property "Value" "GND"
+			(at 27.94 74.93 0)
+			(effects
+				(font
+					(size 1.27 1.27)
+				)
+			)
+		)
+		(property "Footprint" ""
+			(at 27.94 69.85 0)
+			(effects
+				(font
+					(size 1.27 1.27)
+				)
+				(hide yes)
+			)
+		)
+		(property "Datasheet" ""
+			(at 27.94 69.85 0)
+			(effects
+				(font
+					(size 1.27 1.27)
+				)
+				(hide yes)
+			)
+		)
+		(property "Description" "Power symbol creates a global label with name \"GND\" , ground"
+			(at 27.94 69.85 0)
+			(effects
+				(font
+					(size 1.27 1.27)
+				)
+				(hide yes)
+			)
+		)
+		(pin "1"
+		)
+		(instances
+			(project ""
+				(path "/9d05689f-cd28-4719-8892-8398308a18b8"
+					(reference "#PWR010")
+					(unit 1)
+				)

Commit message: update
Parts:
- removed TP1: CC2_TP, TestPoint:TestPoint_Pad_1.0x1.0mm, symbol Connector:TestPoint_Small
- removed TP2: VCONN_TP, TestPoint:TestPoint_Pad_1.0x1.0mm, symbol Connector:TestPoint_Small
- removed TP3: CC1_TP, TestPoint:TestPoint_Pad_1.0x1.0mm, symbol Connector:TestPoint_Small
- removed TP4: GND_TP, TestPoint:TestPoint_Pad_1.0x1.0mm, symbol Connector:TestPoint_Small
- added J6: VBUS_JP, Connector_PinHeader_2.54mm:PinHeader_1x02_P2.54mm_Vertical, symbol Connector:Conn_01x02_Pin
- added J7: VCONN_JP, Connector_PinHeader_2.54mm:PinHeader_1x02_P2.54mm_Vertical, symbol Connector:Conn_01x02_Pin
Connections:
- net +3.3V: now also D5.1 (K), D6.1 (K)
- net GND: now also J6.2 (Pin_2), J7.2 (Pin_2)
- net VCONN: now also J7.1 (Pin_1)
- net VBUS_IN renamed VBUS
- net VBUS: now also J6.1 (Pin_1); no longer D5.1 (K), D6.1 (K)

Commit message: update
Parts:
- removed J2: Dead_Battery_CC1, Connector_PinHeader_2.54mm:PinHeader_1x02_P2.54mm_Vertical, symbol Connector:Conn_01x02_Pin
- removed J3: Dead_Battery_CC2, Connector_PinHeader_2.54mm:PinHeader_1x02_P2.54mm_Vertical, symbol Connector:Conn_01x02_Pin
- removed R5, R6: 5.1k, Resistor_SMD:R_0402_1005Metric, symbol Device:R_Small
- added J2: CC1_TP, Connector_PinHeader_2.54mm:PinHeader_1x01_P2.54mm_Vertical, symbol Connector:Conn_01x01_Pin
- added J3: CC2_TP, Connector_PinHeader_2.54mm:PinHeader_1x01_P2.54mm_Vertical, symbol Connector:Conn_01x01_Pin
Connections:
- net CC1: now also C5.1, J2.1 (Pin_1); no longer C7.1
- net CC2: now also C7.2, J3.1 (Pin_1); no longer C5.1
- net GND: now also C7.1; no longer C7.2
Other:
- moved on the sheet: C5, C7

Commit message: update
Parts:
- added J8: VIN_ENA_JP, Connector_PinHeader_2.54mm:PinHeader_1x02_P2.54mm_Vertical, symbol Connector:Conn_01x02_Pin
Connections:
- net VIN: now reaches C19.1, D3.1 (K), D4.1 (K), U2.7 (VIN)
- net VIN: now also J8.1 (Pin_1)
- net VIN_ENA: now reaches U2.5 (ENA)
- net VIN_ENA: now also J8.2 (Pin_2)
- no-connect marks 29 -> 28
Changed lines of the file:
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@@
 	)
 	(junction
+		(at 41.91 121.92)
+		(diameter 0)
+		(color 0 0 0 0)
+	)
+	(junction
 		(at 238.76 123.19)
 		(diameter 0)
@@
 	)
 	(junction
-		(at 45.72 121.92)
-		(diameter 0)
-		(color 0 0 0 0)
-	)
-	(junction
 		(at 50.8 45.72)
 		(diameter 0)
@@
 	)
 	(no_connect
-		(at 49.53 127)
-	)
-	(no_connect
 		(at 256.54 59.69)
 	)
@@
 	(wire
 		(pts
+			(xy 146.05 137.16) (xy 148.59 137.16)
+		)
+		(stroke
+			(width 0)
+			(type default)
+		)
+	)
+	(wire
+		(pts
 			(xy 27.94 110.49) (xy 27.94 111.76)
 		)
@@
 	(wire
 		(pts
-			(xy 34.29 121.92) (xy 45.72 121.92)
+			(xy 34.29 121.92) (xy 41.91 121.92)
 		)
 		(stroke
@@
 	(wire
 		(pts
-			(xy 45.72 121.92) (xy 49.53 121.92)
-		)
-		(stroke
-			(width 0)
-			(type default)
-		)
-	)
-	(wire
-		(pts
 			(xy 195.58 132.08) (xy 195.58 129.54)
 		)
@@
 	(wire
 		(pts
+			(xy 49.53 127) (xy 48.26 127)
+		)
+		(stroke
+			(width 0)
+			(type default)
+		)
+	)
+	(wire
+		(pts
 			(xy 175.26 27.94) (xy 177.8 27.94)
 		)
@@
 	(wire
 		(pts
+			(xy 146.05 134.62) (xy 148.59 134.62)
+		)
+		(stroke
+			(width 0)
+			(type default)
+		)
+	)
+	(wire
+		(pts
 			(xy 102.87 147.32) (xy 110.49 147.32)
 		)
@@
 	(wire
 		(pts
+			(xy 41.91 121.92) (xy 49.53 121.92)
+		)
+		(stroke
+			(width 0)
+			(type default)
+		)
+	)
+	(wire
+		(pts
 			(xy 238.76 124.46) (xy 238.76 123.19)
 		)
@@
 		)
 	)
+	(label "VIN"
+		(at 148.59 134.62 0)
+		(effects
+			(font
+				(size 1.016 1.016)
+			)
+			(justify left bottom)
+		)
+	)
 	(label "I2C_SDA"
 		(at 205.74 95.25 180)
@@
 		)
 	)
+	(label "VIN"
+		(at 48.26 121.92 180)
+		(effects
+			(font
+				(size 1.016 1.016)
+			)
+			(justify right bottom)
+		)
+	)
 	(label "VBUS"
 		(at 27.94 110.49 180)
@@
 		)
 	)
+	(label "VIN_ENA"
+		(at 148.59 137.16 0)
+		(effects
+			(font
+				(size 1.016 1.016)
+			)
+			(justify left bottom)
+		)
+	)
 	(label "VBUS"
 		(at 111.76 36.83 0)
@@
 		)
 	)
+	(label "VIN_ENA"
+		(at 48.26 127 180)
+		(effects
+			(font
+				(size 1.016 1.016)
+			)
+			(justify right bottom)
+		)
+	)
 	(label "UART_TX"
 		(at 256.54 54.61 0)
@@
 	)
 	(symbol
+		(lib_id "Connector:Conn_01x02_Pin")
+		(at 140.97 134.62 0)
+		(unit 1)
+		(exclude_from_sim no)
+		(in_bom yes)
+		(on_board yes)
+		(dnp no)
+		(property "Reference" "J8"
+			(at 141.605 129.54 0)
+			(effects
+				(font
+					(size 1.27 1.27)
+				)
+			)
+		)
+		(property "Value" "VIN_ENA_JP"
+			(at 140.716 131.572 0)
+			(effects
+				(font
+					(size 0.889 0.889)
+				)
+			)
+		)
+		(property "Footprint" "Connector_PinHeader_2.54mm:PinHeader_1x02_P2.54mm_Vertical"
+			(at 140.97 134.62 0)
+			(effects
+				(font
+					(size 1.27 1.27)
+				)
+				(hide yes)
+			)
+		)
+		(property "Datasheet" "~"
+			(at 140.97 134.62 0)
+			(effects
+				(font
+					(size 1.27 1.27)
+				)
+				(hide yes)
+			)
+		)
+		(property "Description" "Generic connector, single row, 01x02, script generated"
+			(at 140.97 134.62 0)
+			(effects
+				(font
+					(size 1.27 1.27)
+				)
+				(hide yes)
+			)
+		)
+		(pin "1"
+		)
+		(pin "2"
+		)
+		(instances
+			(project ""
+				(path "/9d05689f-cd28-4719-8892-8398308a18b8"
+					(reference "J8")
+					(unit 1)
+				)
+			)
+		)
+	)
+	(symbol
 		(lib_id "Device:C_Small")
 		(at 205.74 34.29 0)
@@
 	(symbol
 		(lib_id "power:PWR_FLAG")
-		(at 45.72 121.92 0)
+		(at 41.91 121.92 0)
 		(unit 1)
 		(exclude_from_sim no)
@@
 		(dnp no)
 		(property "Reference" "#FLG01"
-			(at 45.72 120.015 0)
+			(at 41.91 120.015 0)
 			(effects
 				(font
@@
 		)
 		(property "Value" "PWR_FLAG"
-			(at 45.72 117.856 0)
+			(at 41.91 117.856 0)
 			(effects
 				(font
@@
 		)
 		(property "Footprint" ""
-			(at 45.72 121.92 0)
+			(at 41.91 121.92 0)
 			(effects
 				(font
@@
 		)
 		(property "Datasheet" "~"
-			(at 45.72 121.92 0)
+			(at 41.91 121.92 0)
 			(effects
 				(font
@@
 		)
 		(property "Description" "Special symbol for telling ERC where power comes from"
-			(at 45.72 121.92 0)
+			(at 41.91 121.92 0)
 			(effects
 				(font

Commit message: update
Parts:
- removed J8: VIN_ENA_JP, Connector_PinHeader_2.54mm:PinHeader_1x02_P2.54mm_Vertical, symbol Connector:Conn_01x02_Pin
Connections:
- net VIN_ENA is gone; now on an unnamed net: U2.5 (ENA)
- net VIN: no longer names the net of C19.1, D3.1 (K), D4.1 (K), U2.7 (VIN)

Commit message: update
Parts:
- added J8: VIN_ENA_JP, Connector_PinHeader_2.54mm:PinHeader_1x02_P2.54mm_Vertical, symbol Connector:Conn_01x02_Pin
Connections:
- net VIN: now reaches C19.1, D3.1 (K), D4.1 (K), U2.7 (VIN)
- net VIN: now also J8.1 (Pin_1); no longer U2.5 (ENA)
- new net VIN_ENA: J8.2 (Pin_2), U2.5 (ENA)
Changed lines of the file:
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@@
-	)
-	(junction
-		(at 48.26 121.92)
-		(diameter 0)
-		(color 0 0 0 0)
 	)
 	(junction
@@
 	(wire
 		(pts
+			(xy 146.05 137.16) (xy 148.59 137.16)
+		)
+		(stroke
+			(width 0)
+			(type default)
+		)
+	)
+	(wire
+		(pts
 			(xy 27.94 110.49) (xy 27.94 111.76)
 		)
@@
 	(wire
 		(pts
-			(xy 48.26 121.92) (xy 49.53 121.92)
-		)
-		(stroke
-			(width 0)
-			(type default)
-		)
-	)
-	(wire
-		(pts
 			(xy 82.55 40.64) (xy 110.49 40.64)
 		)
@@
 	(wire
 		(pts
+			(xy 49.53 127) (xy 48.26 127)
+		)
+		(stroke
+			(width 0)
+			(type default)
+		)
+	)
+	(wire
+		(pts
 			(xy 175.26 27.94) (xy 177.8 27.94)
 		)
@@
 	(wire
 		(pts
-			(xy 48.26 127) (xy 48.26 121.92)
-		)
-		(stroke
-			(width 0)
-			(type default)
-		)
-	)
-	(wire
-		(pts
-			(xy 49.53 127) (xy 48.26 127)
-		)
-		(stroke
-			(width 0)
-			(type default)
-		)
-	)
-	(wire
-		(pts
 			(xy 82.55 167.64) (xy 93.98 167.64)
 		)
@@
 	(wire
 		(pts
+			(xy 146.05 134.62) (xy 148.59 134.62)
+		)
+		(stroke
+			(width 0)
+			(type default)
+		)
+	)
+	(wire
+		(pts
 			(xy 102.87 147.32) (xy 110.49 147.32)
 		)
@@
 	(wire
 		(pts
-			(xy 41.91 121.92) (xy 48.26 121.92)
+			(xy 41.91 121.92) (xy 49.53 121.92)
 		)
 		(stroke
@@
 		)
 	)
+	(label "VIN"
+		(at 148.59 134.62 0)
+		(effects
+			(font
+				(size 1.016 1.016)
+			)
+			(justify left bottom)
+		)
+	)
 	(label "I2C_SDA"
 		(at 205.74 95.25 180)
@@
 		)
 	)
+	(label "VIN"
+		(at 48.26 121.92 180)
+		(effects
+			(font
+				(size 1.016 1.016)
+			)
+			(justify right bottom)
+		)
+	)
 	(label "VBUS"
 		(at 27.94 110.49 180)
@@
 		)
 	)
+	(label "VIN_ENA"
+		(at 148.59 137.16 0)
+		(effects
+			(font
+				(size 1.016 1.016)
+			)
+			(justify left bottom)
+		)
+	)
 	(label "VBUS"
 		(at 111.76 36.83 0)
@@
 			)
 			(justify left bottom)
+		)
+	)
+	(label "VIN_ENA"
+		(at 48.26 127 180)
+		(effects
+			(font
+				(size 1.016 1.016)
+			)
+			(justify right bottom)
 		)
 	)
@@
 					(unit 1)
 				)
+			)
+		)
+	)
+	(symbol
+		(lib_id "Connector:Conn_01x02_Pin")
+		(at 140.97 134.62 0)
+		(unit 1)
+		(exclude_from_sim no)
+		(in_bom yes)
+		(on_board yes)
+		(dnp no)
+		(property "Reference" "J8"
+			(at 141.605 129.54 0)
+			(effects
+				(font
+					(size 1.27 1.27)
+				)
+			)
+		)
+		(property "Value" "VIN_ENA_JP"
+			(at 140.716 131.572 0)
+			(effects
+				(font
+					(size 0.889 0.889)
+				)
+			)
+		)
+		(property "Footprint" "Connector_PinHeader_2.54mm:PinHeader_1x02_P2.54mm_Vertical"
+			(at 140.97 134.62 0)
+			(effects
+				(font
+					(size 1.27 1.27)
+				)
+				(hide yes)
+			)
+		)
+		(property "Datasheet" "~"
+			(at 140.97 134.62 0)
+			(effects
+				(font
+					(size 1.27 1.27)
+				)
+				(hide yes)
+			)
+		)
+		(property "Description" "Generic connector, single row, 01x02, script generated"
+			(at 140.97 134.62 0)
+			(effects
+				(font
+					(size 1.27 1.27)
+				)
+				(hide yes)
+			)
+		)
+		(pin "1"
+		)
+		(pin "2"
+		)
+		(instances
+			(project ""
+				(path "/9d05689f-cd28-4719-8892-8398308a18b8"
+					(reference "J8")
+					(unit 1)
+				)
